File: schematic/dip_hat_trick.sch (EAGLE design)
At the start: 12 parts, among them IC2 DS2432P, X1 RPi

Commit message: Update to the DS2431 per info from @KoljaWindeler, Adding pdfs of the Schematic and PCB
Parts:
- removed IC2: DS2432P, 1wire:DS2432P
- added U1: DS2431P, JKW_CHIP:DS2431P
Connections:
- net GND: now also U1.GND; no longer IC2P.GND
- net LCD-D2: now also U1.IO; no longer IC2_1W.1W
Changed lines of the file:
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@@
 <layer number="112" name="tSilk" color="7" fill="1" visible="yes" active="yes"/>
 <layer number="113" name="IDFDebug" color="7" fill="1" visible="yes" active="yes"/>
+<layer number="114" name="Badge_Outline" color="7" fill="1" visible="yes" active="yes"/>
+<layer number="115" name="ReferenceISLANDS" color="7" fill="1" visible="yes" active="yes"/>
 <layer number="116" name="Patch_BOT" color="9" fill="4" visible="yes" active="yes"/>
 <layer number="118" name="Rect_Pads" color="7" fill="1" visible="no" active="no"/>
@@
 <layer number="154" name="FabDoc2" color="7" fill="1" visible="yes" active="yes"/>
 <layer number="155" name="FabDoc3" color="7" fill="1" visible="yes" active="yes"/>
+<layer number="156" name="tAssmbl" color="7" fill="1" visible="yes" active="yes"/>
+<layer number="157" name="bAssmbl" color="7" fill="1" visible="yes" active="yes"/>
 <layer number="199" name="Contour" color="7" fill="1" visible="yes" active="yes"/>
 <layer number="200" name="200bmp" color="1" fill="10" visible="yes" active="yes"/>
@@
 <part name="JP3" library="jumper" deviceset="JP2E" device=""/>
 <part name="GND11" library="supply1" deviceset="GND" device=""/>
-<part name="IC2" library="1wire" deviceset="DS2432" device="P"/>
 <part name="GND14" library="supply1" deviceset="GND" device=""/>
 <part name="R1" library="rcl" deviceset="R-EU_" device="R0805"/>
@@
 <part name="GND5" library="wirepad" deviceset="WIREPAD" device="3,17/1,3"/>
 <part name="X1" library="con-samtec" deviceset="SSW-120-02-S-D" device="" value="RPi"/>
+<part name="U1" library="JKW_CHIP" deviceset="DS2431" device="P"/>
 </parts>
 <sheets>
@@
 <instance part="JP3" gate="1" x="-38.1" y="254"/>
 <instance part="GND11" gate="1" x="-7.62" y="281.94"/>
-<instance part="IC2" gate="G$1" x="101.6" y="271.78"/>
-<instance part="IC2" gate="P" x="109.22" y="261.62" rot="R270"/>
-<instance part="IC2" gate="_1W" x="106.68" y="264.16"/>
-<instance part="GND14" gate="1" x="99.06" y="256.54"/>
+<instance part="GND14" gate="1" x="99.06" y="284.48" rot="R180"/>
 <instance part="R1" gate="G$1" x="86.36" y="271.78" rot="R90"/>
 <instance part="P+3" gate="VCC" x="86.36" y="281.94" smashed="yes">
@@
 <instance part="X1" gate="-39" x="124.46" y="157.48"/>
 <instance part="X1" gate="-40" x="144.78" y="157.48"/>
+<instance part="U1" gate="G$1" x="116.84" y="276.86" rot="R270"/>
 </instances>
 <busses>
@@
 </segment>
 <segment>
-<pinref part="IC2" gate="P" pin="GND"/>
-<pinref part="GND14" gate="1" pin="GND"/>
-<wire x1="101.6" y1="261.62" x2="99.06" y2="261.62" width="0.1524" layer="91"/>
-<wire x1="99.06" y1="261.62" x2="99.06" y2="259.08" width="0.1524" layer="91"/>
-</segment>
-<segment>
 <pinref part="GND5" gate="G$1" pin="P"/>
 <pinref part="GND11" gate="1" pin="GND"/>
@@
 <label x="63.5" y="167.64" size="1.778" layer="95"/>
 <wire x1="60.96" y1="167.64" x2="68.58" y2="167.64" width="0.1524" layer="91"/>
+</segment>
+<segment>
+<pinref part="U1" gate="G$1" pin="GND"/>
+<wire x1="104.14" y1="279.4" x2="99.06" y2="279.4" width="0.1524" layer="91"/>
+<pinref part="GND14" gate="1" pin="GND"/>
+<wire x1="99.06" y1="279.4" x2="99.06" y2="281.94" width="0.1524" layer="91"/>
 </segment>
 </net>
@@
 </segment>
 <segment>
-<pinref part="IC2" gate="_1W" pin="1W"/>
 <label x="91.44" y="264.16" size="1.778" layer="95"/>
-<wire x1="101.6" y1="264.16" x2="86.36" y2="264.16" width="0.1524" layer="91"/>
+<wire x1="119.38" y1="264.16" x2="86.36" y2="264.16" width="0.1524" layer="91"/>
 <pinref part="R1" gate="G$1" pin="1"/>
 <wire x1="86.36" y1="264.16" x2="81.28" y2="264.16" width="0.1524" layer="91"/>
 <wire x1="86.36" y1="266.7" x2="86.36" y2="264.16" width="0.1524" layer="91"/>
 <junction x="86.36" y="264.16"/>
-</segment>
-</net>
+<pinref part="U1" gate="G$1" pin="IO"/>
+<wire x1="119.38" y1="266.7" x2="119.38" y2="264.16" width="0.1524" layer="91"/>
+</segment>
+</net>
